Commit message: changed dimensions of gripper

File: models/ur5/ur5_and_gripper.urdf.xacro (robot description, xacro)
@@ -298,14 +298,14 @@
       <visual>
         <geometry>
-          <cylinder length="0.053" radius="0.0375"/>
+          <cylinder length="0.085" radius="0.0375"/>
         </geometry>
         <material name="blue"/>
-        <origin rpy="0 1.57075 0" xyz="0.028 0 0"/>
-      </visual>
-      <collision>
-        <geometry>
-          <cylinder length="0.053" radius="0.0375"/>
-        </geometry>
-        <origin rpy="0 1.57075 0" xyz="0.028 0 0"/>
+        <origin rpy="0 1.57075 0" xyz="0.04625 0 0"/>
+      </visual>
+      <collision>
+        <geometry>
+          <cylinder length="0.085" radius="0.0375"/>
+        </geometry>
+        <origin rpy="0 1.57075 0" xyz="0.04625 0 0"/>
       </collision>
       <inertial>
@@ -322,14 +322,14 @@
       <visual>
         <geometry>
-          <box size="0.07 0.025 0.02"/>
+          <box size="0.11 0.025 0.02"/>
         </geometry>
         <material name="blue"/>
-        <origin rpy="0 0 0" xyz="0 0.025 0"/>
-      </visual>
-      <collision>
-        <geometry>
-          <box size="0.07 0.025 0.02"/>
-        </geometry>
-        <origin rpy="0 0 0" xyz="0 0.025 0"/>
+        <origin rpy="0 0 0" xyz="0.055 0.025 0"/>
+      </visual>
+      <collision>
+        <geometry>
+          <box size="0.11 0.025 0.02"/>
+        </geometry>
+        <origin rpy="0 0 0" xyz="0.055 0.025 0"/>
       </collision>
       <inertial>
@@ -346,14 +346,14 @@
       <visual>
         <geometry>
-          <box size="0.07 0.025 0.02"/>
+          <box size="0.11 0.025 0.02"/>
         </geometry>
         <material name="blue"/>
-        <origin rpy="0 0 0" xyz="0 -0.025 0"/>
-      </visual>
-      <collision>
-        <geometry>
-          <box size="0.07 0.025 0.02"/>
-        </geometry>
-        <origin rpy="0 0 0" xyz="0 -0.025 0"/>
+        <origin rpy="0 0 0" xyz="0.055 -0.025 0"/>
+      </visual>
+      <collision>
+        <geometry>
+          <box size="0.11 0.025 0.02"/>
+        </geometry>
+        <origin rpy="0 0 0" xyz="0.055 -0.025 0"/>
       </collision>
       <inertial>
